Commit message: update car urdf model

File: robocar_ws/src/robo_car/world/prius_hybrid/car.urdf (robot description, URDF)
Before this commit: robot prius_hybrid, 3 links, 2 joints
Links:
- added link camera_link_optical
- added link rear_axle
- added link rear_left_wheel
- added link rear_right_wheel
Joints:
- added joint camera_joint: type fixed, parent sensors, child front_camera_sensor, origin xyz=0 -0.4 1.4 rpy=0 0.05 -1.5707
- added joint rear_axle_joint: type fixed, parent chassis, child rear_axle, origin xyz=0 1.45 0.3 rpy=0 0 0
- added joint rear_left_wheel_joint: type fixed, parent rear_axle, child rear_left_wheel, origin xyz=0.786 1.45 0.3 rpy=0 0 0
- added joint rear_right_wheel_joint: type fixed, parent rear_axle, child rear_right_wheel, origin xyz=-0.786 1.45 0.3 rpy=0 0 0
- joint camera_optical_joint: child front_camera_sensor -> camera_link_optical; origin xyz=0 -0.4 1.4 rpy=0 0.05 -1.5707 -> xyz=0 0 0 rpy=-1.5707 0 -1.5707; parent sensors -> front_camera_sensor

Commit message: update car model and git submodule

File: robocar_ws/src/robo_car/world/prius_hybrid/car.urdf (robot description, URDF)
Before this commit: robot prius_hybrid, 7 links, 6 joints
Links:
- added link front_left_wheel
- added link front_right_wheel
- link chassis: geometry 
Joints:
- added joint front_left_combined_joint: type fixed, parent chassis, child front_left_wheel, origin xyz=0.6727335374 -1.41 0.3 rpy=0 0 0
- added joint front_right_combined_joint: type fixed, parent chassis, child front_right_wheel, origin xyz=-0.8472664626 -1.41 0.3 rpy=0 0 0
